File: Circuits/power_control_circuit_V1/Power Control Circuit.kicad_sch (KiCad schematic)
At the start: 37 parts, among them Q1 S8050, Q21 S8050, Q23 S8050, Q24 S8550, Q25 IRF3205, Q3 S8050, Q4 S8550, Q5 IRF3205, Q6 IRF3205, Q7 IRF3205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

Commit message: Major circuit changes and LCD driver finished and tested
Parts:
- removed LCD1: Conn_01x16_Female, Connector_PinSocket_2.54mm:PinSocket_1x16_P2.54mm_Vertical, symbol circuit-rescue:Conn_01x16_Female-Connector
- removed Switch1, Switch2: Switchhhhhh, Resistor_THT:R_Axial_DIN0204_L3.6mm_D1.6mm_P5.08mm_Vertical, symbol Device:R
- added DS1: WC1602A, Display:WC1602A, symbol Display_Character:WC1602A
- added SW1, SW2: SW_MEC_5E, Button_Switch_THT:SW_PUSH-12mm, symbol Switch:SW_MEC_5E
- added U1, U2: PC817, Package_DIP:DIP-4_W7.62mm, symbol Isolator:PC817
- R11, R13, R15: value 330 -> 1k
- R12, R14, R16: value 10,000 -> 10k
- R18: value 1,000 -> 330
Connections:
- net +5V: now also R18.1, DS1.2 (VDD)
- net Charging: now also Microcontroller1.12 (RB6/T1OSC0/T1CKI/PGC); no longer Microcontroller1.16 (CLKIN/OSC1/RA7)
- net D4: now also Microcontroller1.6 (RB0/INT), DS1.11 (D4); no longer Microcontroller1.8 (RB2/TX/CK)
- net D5: now also Microcontroller1.7 (RB1/RX/DT), DS1.12 (D5); no longer Microcontroller1.9 (RB3/CCP1)
- net D6: now also Microcontroller1.8 (RB2/TX/CK), DS1.13 (D6); no longer Microcontroller1.10 (RB4/PGM)
- net D7: now also Microcontroller1.9 (RB3/CCP1), DS1.14 (D7); no longer Microcontroller1.11 (RB5)
- net Discharge: now also Microcontroller1.13 (RB7/T1OSI/PGD); no longer Microcontroller1.15 (CLKOUT/OSC2/RA6)
- net EN: now also Microcontroller1.10 (RB4/PGM), DS1.6 (E); no longer Microcontroller1.7 (RB1/RX/DT)
- net GND: now also DS1.1 (VSS), DS1.16 (LED(-)), DS1.5 (R/W); no longer R18.2
- net RS: now also Microcontroller1.11 (RB5), DS1.4 (RS); no longer Microcontroller1.6 (RB0/INT)
- net arrowkey: now also Microcontroller1.4 (~{MCLR}/Vpp/RA5), SW1.4 (A); no longer Microcontroller1.13 (RB7/T1OSI/PGD)
- net enterkey: now also Microcontroller1.15 (CLKOUT/OSC2/RA6), SW2.4 (A); no longer Microcontroller1.12 (RB6/T1OSC0/T1CKI/PGC)
- net weldingkey: now also Microcontroller1.16 (CLKIN/OSC1/RA7); no longer Microcontroller1.17 (AN0/RA0)
- net at R13.2: now also SW2.1
- net at LCDcontrastTrimmer1.2: now also DS1.3 (VO)
- net at R11.2: now also SW1.1
- new net: DS1.15 (LED(+)), R18.2
Other:
- moved on the sheet: LCDcontrastTrimmer1, R12, R14
