File: Circuits/power_control_circuit_V2/Power Control Circuit.kicad_sch (KiCad schematic)
At the start: 36 parts, among them Q10 IRF1405, Q12 IRF1405, Q23 S8050, Q24 S8550, Q3 S8050, Q4 IRF1405, Q4 S8550, Q8 IRF1405, Q9 IRF1405, SW1 SW_MEC_5E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

Commit message: finished Middle and application layer
Parts:
- removed Button1: AudioJack2, Connector_Audio:Jack_3.5mm_CUI_SJ-3523-SMT_Horizontal, symbol circuit-rescue:AudioJack2-Connector
- removed R10: 510,000, Resistor_THT:R_Axial_DIN0207_L6.3mm_D2.5mm_P7.62mm_Horizontal, symbol Device:R
- removed R9: 1,000, Resistor_THT:R_Axial_DIN0207_L6.3mm_D2.5mm_P7.62mm_Horizontal, symbol Device:R
- removed SW1, SW2: SW_MEC_5E, Button_Switch_THT:SW_PUSH-12mm, symbol Switch:SW_MEC_5E
- added ARROW_BUTTON, ENTER_BUTTON, WELD_BUTTON: Conn_01x02_Socket, symbol Connector:Conn_01x02_Socket
- added LCD_OUT: Conn_01x12_Socket, Connector_PinHeader_2.54mm:PinHeader_1x12_P2.54mm_Vertical, symbol Connector:Conn_01x12_Socket
Connections:
- net +5V: now also LCD_OUT.2 (Pin_2)
- net D4: now also LCD_OUT.7 (Pin_7)
- net D5: now also LCD_OUT.8 (Pin_8)
- net D6: now also LCD_OUT.9 (Pin_9)
- net D7: now also LCD_OUT.10 (Pin_10)
- net EN: now also LCD_OUT.6 (Pin_6)
- net GND: now also LCD_OUT.1 (Pin_1), LCD_OUT.12 (Pin_12), LCD_OUT.5 (Pin_5)
- net RS: now also LCD_OUT.4 (Pin_4)
- net arrowkey: now also ARROW_BUTTON.1 (Pin_1)
- net enterkey: now also ENTER_BUTTON.1 (Pin_1)
- net weldingkey: now also WELD_BUTTON.1 (Pin_1)
- net at R13.2: now also ENTER_BUTTON.2 (Pin_2)
- net LED+: now reaches DS1.15 (LED(+)), R18.2
- net LED+: now also LCD_OUT.11 (Pin_11)
- net VO: now reaches DS1.3 (VO), LCDcontrastTrimmer1.2
- net VO: now also LCD_OUT.3 (Pin_3)
- net at R11.2: now also ARROW_BUTTON.2 (Pin_2)
- net at R15.2: now also WELD_BUTTON.2 (Pin_2)
- net VoltageDividerRef: no longer names the net of Microcontroller1.18 (AN1/RA1)
Other:
- moved on the sheet: DS1, LCDcontrastTrimmer1, R18
