File: Circuits/power_control_circuit_V2/final_version/Power Control Circuit.kicad_pcb (KiCad board)
At the start: 2 copper layers, 33 parts, among them Q10 IRF1405, Q12 IRF1405, Q2 S8050, Q3 S8550, Q4 IRF1405, Q6 S8050, Q7 S8550, Q8 IRF1405, Q9 IRF1405, U1 PC817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

Commit message: further development in V2 final version
Parts:
- moved LCDcontrastTrimmer1 136.1 mm to (41.4, 143.8), turned to 90 degrees
- moved ARROW_BUTTON1 120.0 mm to (48.1, 130.2), turned to 90 degrees
- moved uC_Power_input1 108.8 mm to (58.4, 118.8), turned to 180 degrees
- moved ENTER_BUTTON1 103.8 mm to (63.6, 130.1), turned to 90 degrees
- moved WELD_BUTTON1 103.1 mm to (63.6, 121.6), turned to 90 degrees
- moved Microcontroller1 101.9 mm to (52.3, 122.6)
- moved Q2 94.8 mm to (86.1, 145.9), turned to -90 degrees
- moved U2 92.5 mm to (72.3, 140.4)
- moved U1 92.5 mm to (72.3, 134.7)
- moved Q3 91.4 mm to (86.8, 143.0), turned to 90 degrees
- moved Q7 88.8 mm to (86.1, 135.0), turned to -90 degrees
- moved Q6 88.3 mm to (86.8, 132.0), turned to 90 degrees
- moved LCD_OUT1 87.2 mm to (38.3, 148.2), turned to 90 degrees
- moved R6 68.5 mm to (37.3, 126.2)
- moved R7 60.9 mm to (45.0, 131.7), turned to 180 degrees
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Routing:
- net GND: track 0.00 -> 170.1 mm
- net +5V: track 0.00 -> 137.4 mm
- net RS: track 0.00 -> 42.6 mm
- net EN: track 0.00 -> 33.2 mm
- net +12V: track 0.00 -> 30.5 mm
- net D4: track 0.00 -> 17.3 mm
- net GNDA: track 0.00 -> 16.9 mm
- net D5: track 0.00 -> 16.3 mm
- net Net-(Q2-E): track 0.00 -> 15.1 mm
- net Net-(Q6-B): track 0.00 -> 15.0 mm
- net Net-(Q2-B): track 0.00 -> 14.4 mm
- net D6: track 0.00 -> 14.0 mm
- net weldingkey: track 0.00 -> 12.0 mm
- net D7: track 0.00 -> 11.0 mm
- net enterkey: track 0.00 -> 8.07 mm
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
Commit message: finished PCB final version :)
Parts:
- added HS1: Heatsink_Pad_2Pin, Heatsink:Heatsink_Stonecold_HS-S03_13.21x12.7mm, F.Cu at (141.8, 132.0)
- added HS2: Heatsink_Pad_2Pin, Heatsink:Heatsink_Stonecold_HS-S03_13.21x12.7mm, F.Cu at (103.2, 145.7)
- added HS3: Heatsink_Pad_2Pin, Heatsink:Heatsink_Stonecold_HS-S03_13.21x12.7mm, F.Cu at (125.4, 132.0)
- added HS4: Heatsink_Pad_2Pin, Heatsink:Heatsink_Stonecold_HS-S03_13.21x12.7mm, F.Cu at (109.0, 132.0)
- added HS5: Heatsink_Pad_2Pin, Heatsink:Heatsink_Stonecold_HS-S03_13.21x12.7mm, F.Cu at (92.6, 131.9)
- moved Q8 42.3 mm to (140.0, 129.5), turned to -90 degrees
- moved Rsense1 33.5 mm to (108.6, 145.1)
- moved Q12 25.5 mm to (90.7, 129.4), turned to -90 degrees
- moved Q9 20.2 mm to (123.5, 129.5), turned to -90 degrees
- moved Electrodes1 13.8 mm to (141.4, 121.2), turned to 180 degrees
- moved CapacitorBank1 12.8 mm to (146.9, 121.2)
- moved PowerInput1 9.87 mm to (143.8, 145.2)
- moved Q4 7.32 mm to (105.2, 147.8)
- moved Q10 5.50 mm to (107.1, 129.4), turned to -90 degrees
Routing:
- net +12V: track 30.5 -> 148.1 mm
- net GNDS: track 0.00 -> 117.0 mm
- net Net-(Electrodes1-Pin_1): track 0.00 -> 67.9 mm
- net GNDA: track 16.9 -> 79.9 mm
- net Net-(Q10-G): track 3.24 -> 56.6 mm
- net Net-(Q2-E): track 15.1 -> 22.6 mm
- net Net-(Q4-D): track 0.00 -> 5.17 mm
Other:
- board outline added: 122.3 x 43.4 mm
