File: Circuits/power_control_circuit_V2/final_version/Power Control Circuit.kicad_sch (KiCad schematic)
At the start: 41 parts, among them Q10 IRF1405, Q12 IRF1405, Q23 S8050, Q24 S8550, Q3 S8050, Q4 IRF1405, Q4 S8550, Q8 IRF1405, Q9 IRF1405, U1 PC817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

Commit message: minor changes
Parts:
- added Q1: IRF540N, Package_TO_SOT_THT:TO-220-3_Vertical, symbol Transistor_FET:IRF540N
Changed lines of the file:
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@@
+    )
+  )
+  (symbol (lib_id "Transistor_FET:IRF540N") (at 279.4 73.66 0) (unit 1)
+    (in_bom yes) (on_board yes) (dnp no) (fields_autoplaced)
+    (property "Reference" "Q1" (at 285.75 72.39 0)
+      (effects (font (size 1.27 1.27)) (justify left))
+    )
+    (property "Value" "IRF540N" (at 285.75 74.93 0)
+      (effects (font (size 1.27 1.27)) (justify left))
+    )
+    (property "Footprint" "Package_TO_SOT_THT:TO-220-3_Vertical" (at 284.48 75.565 0)
+      (effects (font (size 1.27 1.27) italic) (justify left) hide)
+    )
+    (property "Datasheet" "http://www.irf.com/product-info/datasheets/data/irf540n.pdf" (at 284.48 77.47 0)
+      (effects (font (size 1.27 1.27)) (justify left) hide)
+    )
+    (pin "3")
+    (pin "2")
+    (pin "1")
+    (instances
+      (project "Power Control Circuit"
+        (path "/f5e3c383-3430-4217-817e-2eedfeb82870"
+          (reference "Q1") (unit 1)
+        )
+      )
     )
   )
